File: 57x80/procyon_57x80.kicad_pcb (KiCad board)
At the start: 4 copper layers, 57.2 x 80 mm, 34 parts, among them J1 Conn_01x07_Pin, Q1 AO3401A, U1 mXT336UD-MAU002

Commit message: Completed routing for 57x80
Parts:
- moved NT1 17.0 mm to (25.2, 111.9)
Connections:
- U1 pad 11: unconnected-(U1-X10-Pad11) -> /X10
- U1 pad 12: unconnected-(U1-X11-Pad12) -> /X11
- U1 pad 13: unconnected-(U1-X12-Pad13) -> /X12
- U1 pad 14: unconnected-(U1-X13-Pad14) -> /X13
- U1 pad 17: unconnected-(U1-Y12-Pad17) -> /Y12
- U1 pad 18: unconnected-(U1-Y13-Pad18) -> /Y13
- U1 pad 19: unconnected-(U1-Y14-Pad19) -> /Y14
- U1 pad 20: unconnected-(U1-Y15-Pad20) -> /Y15
- U1 pad 21: unconnected-(U1-Y16-Pad21) -> /Y16
- U1 pad 22: unconnected-(U1-Y17-Pad22) -> /Y17
- U1 pad 23: unconnected-(U1-Y18-Pad23) -> /Y18
- U1 pad 24: unconnected-(U1-Y19-Pad24) -> /Y19
Routing:
- net /Y19: track 0.00 -> 120.8 mm, vias 0 -> 1
- net /Y18: track 0.00 -> 117.4 mm, vias 0 -> 1
- net /Y17: track 0.00 -> 114.0 mm, vias 0 -> 1
- net /Y16: track 0.00 -> 110.7 mm, vias 0 -> 1
- net /X13: track 0.00 -> 108.8 mm, vias 0 -> 21
- net /Y15: track 0.00 -> 107.4 mm, vias 0 -> 1
- net /X12: track 0.00 -> 105.0 mm, vias 0 -> 21
- net /Y14: track 0.00 -> 104.4 mm, vias 0 -> 1
- net /X11: track 0.00 -> 102.1 mm, vias 0 -> 21
- net /Y13: track 0.00 -> 101.2 mm, vias 0 -> 1
- net /Y12: track 0.00 -> 99.8 mm, vias 0 -> 1
- net /X10: track 0.00 -> 99.1 mm, vias 0 -> 21
- net /X1: track 59.2 -> 105.7 mm, vias 13 -> 21
- net /X2: track 56.8 -> 100.8 mm, vias 13 -> 21
- net /X0: track 64.4 -> 107.7 mm, vias 13 -> 21
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- added copper zone on B.Cu, net /X0
- added copper zone on B.Cu, net /X1
- added copper zone on B.Cu, net /X10
- added copper zone on B.Cu, net /X11
- added copper zone on B.Cu, net /X12
- added copper zone on B.Cu, net /X13
- added copper zone on B.Cu, net /X2
- added copper zone on B.Cu, net /X3
- added copper zone on B.Cu, net /X4
- added copper zone on B.Cu, net /X5
- added copper zone on B.Cu, net /X6
- added copper zone on B.Cu, net /X7
- added copper zone on B.Cu, net /X8
- added copper zone on B.Cu, net /X9
- added copper zone on B.Cu, net /Y0
- added copper zone on B.Cu, net /Y1
- added copper zone on B.Cu, net /Y10
- added copper zone on B.Cu, net /Y11
- added copper zone on B.Cu, net /Y12
- added copper zone on B.Cu, net /Y13
- added copper zone on B.Cu, net /Y14
- added copper zone on B.Cu, net /Y15
- added copper zone on B.Cu, net /Y16
- added copper zone on B.Cu, net /Y17
- added copper zone on B.Cu, net /Y18
- added copper zone on B.Cu, net /Y19
- added copper zone on B.Cu, net /Y2
- added copper zone on B.Cu, net /Y3
- added copper zone on B.Cu, net /Y4
- added copper zone on B.Cu, net /Y5
- added copper zone on B.Cu, net /Y6
- added copper zone on B.Cu, net /Y7
- added copper zone on B.Cu, net /Y8
- added copper zone on B.Cu, net /Y9
- removed copper zone on B.Cu, net (none)
Other:
- board text added: "Procyon (57.2x80mm) v1.00 by George Norton"
- board text removed: "Procyon (49.6x42mm) v1.00 by George Norton"
